File: Exerc_02.sch (KiCad schematic (older format))
At the start: 27 parts, among them P1 JP7, P2 JP6, P3 USB_A, U1 ATmega32U4, U2 MIC5219, Y1 Crystal

Commit message: Finalizado PCB
Parts:
- P3: footprint Connectors:USB_B -> Connectors:USB_Micro-B
Changed lines of the file:
@@
 LIBS:contrib
 LIBS:valves
+LIBS:NorBot
 LIBS:Exerc_02-cache
 EELAYER 25 0
@@
 F 0 "P3" H 4850 3700 50  0000 C CNN
 F 1 "USB_A" H 4600 4100 50  0000 C CNN
-F 2 "Connectors:USB_B" V 4600 3800 50  0001 C CNN
+F 2 "Connectors:USB_Micro-B" V 4600 3800 50  0001 C CNN
 F 3 "" V 4600 3800 50  0000 C CNN
 	1    4650 3900
