File: Exerc_02.kicad_pcb (KiCad board)
At the start: 2 copper layers, 35 x 25 mm, 27 parts, among them P1 JP7, P2 JP6, P3 USB_A, U1 ATmega32U4, U2 MIC5219, Y1 Crystal

Commit message: Finalizado PCB
Parts:
- P3: footprint Connectors:USB_B -> Connectors:USB_Micro-B
- moved D2 81.1 mm to (202.8, 126.0), turned to 180 degrees
- moved R1 66.8 mm to (202.8, 130.2)
- moved C9 62.9 mm to (188.3, 131.6)
- moved C7 62.3 mm to (185.2, 134.3), turned to 180 degrees
- moved R2 57.2 mm to (184.5, 131.1), turned to 180 degrees
- moved C8 53.8 mm to (201.8, 138.4)
- moved C3 50.7 mm to (174.2, 142.0), turned to 180 degrees
- moved D3 50.4 mm to (193.6, 138.3)
- moved R6 50.0 mm to (183.3, 141.9), turned to 180 degrees
- moved D1 49.4 mm to (178.0, 122.4), turned to 180 degrees
- moved C2 46.5 mm to (181.6, 133.2), turned to 270 degrees
- moved C5 46.0 mm to (202.4, 133.9)
- moved R3 45.4 mm to (181.7, 127.6)
- moved Y1 44.1 mm to (173.4, 138.3), turned to 180 degrees
- moved D4 44.1 mm to (179.3, 142.4), turned to 180 degrees
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Connections:
- P1 pad 11: RTX -> (no net)
- P2 pad 3: RESET -> (no net)
- P3 pad 5: Net-(P3-Pad5) -> (no net)
- U1 pad 12: D11 -> (no net)
- U1 pad 20: RX1 -> (no net)
- U1 pad 26: D12 -> (no net)
- U1 pad 3: D- -> (no net)
- U1 pad 32: D13 -> (no net)
- U1 pad 40: A4 -> (no net)
- U1 pad 41: A5 -> (no net)
- U2 pad 4: Net-(U2-Pad4) -> (no net)
Routing:
- net VCC: track 14.2 -> 86.2 mm, vias 2 -> 11
- net Net-(R6-Pad1): track 0.00 -> 32.2 mm, vias 0 -> 4
- net Net-(C8-Pad1): track 0.00 -> 32.1 mm, vias 0 -> 3
- net UVCC: track 0.00 -> 32.0 mm, vias 0 -> 4
- net Net-(C7-Pad1): track 0.00 -> 30.3 mm, vias 0 -> 3
- net GND: track 10.6 -> 35.5 mm, vias 0 -> 8
- net RAW: track 0.00 -> 20.7 mm
- net SCK: track 14.9 -> 33.5 mm, vias 2 -> 4
- net D+: track 0.00 -> 18.0 mm, vias 0 -> 2
- net Net-(R4-Pad1): track 0.00 -> 12.5 mm, vias 0 -> 2
- net Net-(P3-Pad3): track 0.00 -> 12.4 mm, vias 0 -> 2
- net Net-(C9-Pad1): track 0.00 -> 9.79 mm, vias 0 -> 2
- net Net-(P3-Pad2): track 0.00 -> 9.78 mm, vias 0 -> 2
- net MOSI: track 12.1 -> 21.8 mm, vias 0 -> 2
- net Net-(R5-Pad1): track 0.00 -> 9.44 mm, vias 0 -> 2
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- added copper zone on B.Cu, net GND
Other:
- net class Default: clearance 0.2 -> 0.1524
- rule trace_clearance: 0.2 -> 0.1524

Commit message: Atualizado algumas trilhas.
Routing:
- net GND: track 35.5 -> 51.4 mm, vias 8 -> 14
- net VCC: track 86.2 -> 95.2 mm, vias 11 -> 15
- net UVCC: track 32.0 -> 40.0 mm, vias 4 -> 6
- net D+: track 18.0 -> 20.2 mm
- net SCK: track 33.5 -> 31.8 mm
- net MISO: track 21.5 -> 20.3 mm
- net MOSI: track 21.8 -> 22.4 mm
Other:
- net class Default: via_drill 0.4 -> 0.3302
